File: hardware/kicad_regie_hub/regie_hub_mega_esp32.kicad_pcb (KiCad board)
At the start: 2 copper layers, 134 x 80 mm, 12 parts

Commit message: hardware: passifs + petits connecteurs en CMS pour assemblage PCBA
Par choix explicite (assemblage machine chez le fabricant plutot que
soudure manuelle): resistances et condensateurs passent en CMS 0805
(R_0805/C_0805), et les petits connecteurs "fils volants" (bouton, module
de charge, module vibreur, batterie, interrupteur) passent en variantes
SMD des memes footprints PinSocket. Meme numerotation de broche que les
versions traversantes -- NETS inchange, seule l'empreinte change.

Restent traversants (headers de modules enfichables, pas adaptes au CMS):
A1L/A1R (nano), U1L/U1R (esp32), U_ESP32L/R (hub), J1/J_NRF (nRF24),
J_MEGA (hub).

Nano: C1, SW1, SW2, J2, J3, BT1 -> CMS.
ESP32: SW1, SW2, J2, J3, BT1 -> CMS.
Hub: R1-R4, C1-C3 -> CMS.

Les 3 cartes re-routees (Freerouting) et revalidees (kicad-cli pcb drc):
0 violation de clearance, 0 element non connecte, keepout nRF24 toujours
respecte (0 piste dedans, verifie par script), 0 track_dangling apres
nettoyage des residus d'autorouter habituels.

Co-Authored-By: Claude Sonnet 5 <noreply@anthropic.com>
Parts:
- C1: value ~10uF decouplage entree regulateur -> ~10uF decouplage entree regulateur - CMS; footprint Capacitor_THT:C_Disc_D10.5mm_W5.0mm_P5.00mm -> Capacitor_SMD:C_0805_2012Metric
- C2: value ~10uF decouplage sortie regulateur -> ~10uF decouplage sortie regulateur - CMS; footprint Capacitor_THT:C_Disc_D10.5mm_W5.0mm_P5.00mm -> Capacitor_SMD:C_0805_2012Metric
- C3: value 10-100uF decouplage nRF24 (obligatoire, au plus pres) -> 10-100uF decouplage nRF24 (obligatoire, au plus pres) - CMS; footprint Capacitor_THT:C_Disc_D10.5mm_W5.0mm_P5.00mm -> Capacitor_SMD:C_0805_2012Metric
- R1: value 1k (diviseur TX2, serie) -> 1k (diviseur TX2, serie) - CMS; footprint Resistor_THT:R_Axial_DIN0207_L6.3mm_D2.5mm_P7.62mm_Horizontal -> Resistor_SMD:R_0805_2012Metric
- R2: value 2k (diviseur TX2, vers GND) -> 2k (diviseur TX2, vers GND) - CMS; footprint Resistor_THT:R_Axial_DIN0207_L6.3mm_D2.5mm_P7.62mm_Horizontal -> Resistor_SMD:R_0805_2012Metric
- R3: value 1k (diviseur TX3, serie) -> 1k (diviseur TX3, serie) - CMS; footprint Resistor_THT:R_Axial_DIN0207_L6.3mm_D2.5mm_P7.62mm_Horizontal -> Resistor_SMD:R_0805_2012Metric
- R4: value 2k (diviseur TX3, vers GND) -> 2k (diviseur TX3, vers GND) - CMS; footprint Resistor_THT:R_Axial_DIN0207_L6.3mm_D2.5mm_P7.62mm_Horizontal -> Resistor_SMD:R_0805_2012Metric
Routing:
- net GND: track 165.4 -> 205.4 mm, vias 0 -> 1
- net NRF_SCK: track 54.3 -> 41.0 mm, vias 1 -> 0
- net MEGA_RX2_DIRECT: track 68.4 -> 72.7 mm
- net ESP32_RX2_3V3: track 37.9 -> 34.8 mm, vias 0 -> 1
- net NRF_VCC_DEDIE: track 96.3 -> 98.0 mm
- net ESP32_RX1_3V3: track 57.9 -> 59.3 mm, vias 0 -> 1
- net MEGA_TX2_5V: track 20.0 -> 19.1 mm
- net VCC_5V_MEGA: track 123.9 -> 124.3 mm, vias 0 -> 1

Commit message: hardware: carte ESP32 equipe 65x50mm, BOM CSV, libelle J_MEGA hub
ESP32 equipe reduite a 65x50mm (U1L/U1R et J2/J3 pivotes a 90 degres),
reroutee, DRC sans clearance ni connexion manquante. Gerbers regeneres.
Fichiers BOM CSV ajoutes pour les 3 cartes. Hub : libelle J_MEGA
TX1/RX1 (pins 18/19) au lieu de TX3/RX3, sans changement de routage.

Co-Authored-By: Claude Sonnet 5 <noreply@anthropic.com>
Parts:
- J_MEGA: value Vers Mega: TX2 RX2 TX3 RX3 5V GND -> Vers Mega: TX2(16) RX2(17) TX1(18) RX1(19) 5V GND
Changed lines of the file:
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@@
 			)
 		)
-		(property "Value" "Vers Mega: TX2 RX2 TX3 RX3 5V GND"
+		(property "Value" "Vers Mega: TX2(16) RX2(17) TX1(18) RX1(19) 5V GND"
 			(at 0 15.47 0)
 			(layer "F.Fab")
